File: usb-power-delayer/schematic.brd (EAGLE design)
At the start: 100 x 80 mm, 8 parts, among them Q1 BC547B, Q3 BS250

Commit message: [USB-Delayer] Extend the delay time from ~35s to ~52s as 35s was sometimes not enough.
Parts:
- R1: value 68k -> 78k
Changed lines of the file:
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@@
 <attribute name="VALUE" x="21.59" y="20.955" size="1.27" layer="27" ratio="10" rot="R270"/>
 </element>
-<element name="R1" library="rcl" library_urn="urn:adsk.eagle:library:334" package="0204/5" package3d_urn="urn:adsk.eagle:package:23488/1" value="68k" x="33.02" y="25.4" smashed="yes" rot="R270">
+<element name="R1" library="rcl" library_urn="urn:adsk.eagle:library:334" package="0204/5" package3d_urn="urn:adsk.eagle:package:23488/1" value="78k" x="33.02" y="25.4" smashed="yes" rot="R270">
 <attribute name="NAME" x="34.3154" y="27.94" size="0.9906" layer="25" ratio="10" rot="R270"/>
 <attribute name="POPULARITY" value="35" x="-10.16" y="7.62" size="1.778" layer="27" rot="R270" display="off"/>
