File: inverter-welder/concepts/08_magnum_power_vip_4000/improvements/current_setting_display/schematic.brd (EAGLE design)
At the start: 100 x 80 mm, 7 parts, among them P1 1k

Commit message: [Welder] Improve schematic.
Parts:
- moved VR2 17.6 mm to (8.89, 61.6), turned to 0 degrees
- moved VR3 16.8 mm to (15.9, 47.0), turned to 270 degrees
- moved JP1 4.58 mm to (19.1, 57.1)
- moved 15.8V 1.27 mm to (21.6, 36.8)
- moved VR1 0.64 mm to (8.89, 37.5)
Connections:
- net GND: now also VR2.A; no longer VR3.A
- net N$1: now also VR3.A; no longer VR2.A
- net N$2: now also VR3.S; no longer VR2.S
- net N$4: now also VR2.S; no longer VR3.S
Routing:
- net N$2: track 8.04 -> 10.2 mm
- net N$6: track 18.9 -> 17.0 mm
- net N$1: track 8.89 -> 7.73 mm
- net N$3: track 14.4 -> 13.4 mm
- net N$4: track 10.4 -> 9.80 mm
- net N$5: track 9.39 -> 8.75 mm
- net N$8: track 24.2 -> 23.7 mm
