File: inverter-welder/concepts/08_magnum_power_vip_4000/improvements/current_setting_display/schematic.sch (EAGLE design)
At the start: 7 parts, among them P1 1k

Commit message: [Welder] Improve schematic.
Connections:
- net GND: now also VR2.A; no longer VR3.A
- net N$1: now also VR3.A; no longer VR2.A
- net N$2: now also VR3.S; no longer VR2.S
- net N$4: now also VR2.S; no longer VR3.S
Other:
- note added: "do czarnego przewódu nastawy prądu"
- note added: "do czerwonego przewódu nastawy prądu"
- note added: "do zielonego przewódu nastawy prądu"
- moved on the sheet: VR2, VR3
Changed lines of the file:
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@@
 <parts>
 <part name="P1" library="pot" library_urn="urn:adsk.eagle:library:331" deviceset="3RP/1610G" device="" package3d_urn="urn:adsk.eagle:package:22728/1" value="1k"/>
-<part name="VR2" library="pot" library_urn="urn:adsk.eagle:library:331" deviceset="TRIM_EU-" device="RJ9W" package3d_urn="urn:adsk.eagle:package:22702/1" value="500"/>
+<part name="VR3" library="pot" library_urn="urn:adsk.eagle:library:331" deviceset="TRIM_EU-" device="RJ9W" package3d_urn="urn:adsk.eagle:package:22702/1" value="500"/>
 <part name="JP1" library="pinhead" library_urn="urn:adsk.eagle:library:325" deviceset="PINHD-1X3" device="" package3d_urn="urn:adsk.eagle:package:22458/2"/>
 <part name="VR1" library="pot" library_urn="urn:adsk.eagle:library:331" deviceset="TRIM_EU-" device="RJ9W" package3d_urn="urn:adsk.eagle:package:22702/1" value="10k"/>
-<part name="VR3" library="pot" library_urn="urn:adsk.eagle:library:331" deviceset="TRIM_EU-" device="RJ9W" package3d_urn="urn:adsk.eagle:package:22702/1" value="500"/>
+<part name="VR2" library="pot" library_urn="urn:adsk.eagle:library:331" deviceset="TRIM_EU-" device="RJ9W" package3d_urn="urn:adsk.eagle:package:22702/1" value="500"/>
 <part name="GND1" library="supply1" library_urn="urn:adsk.eagle:library:371" deviceset="GND" device=""/>
 <part name="GND2" library="supply1" library_urn="urn:adsk.eagle:library:371" deviceset="GND" device=""/>
@@
 <sheet>
 <plain>
+<text x="116.84" y="53.34" size="1.778" layer="97">do czerwonego przewódu nastawy prądu</text>
+<text x="116.84" y="50.8" size="1.778" layer="97">do czarnego przewódu nastawy prądu</text>
+<text x="116.84" y="48.26" size="1.778" layer="97">do zielonego przewódu nastawy prądu</text>
 </plain>
 <instances>
@@
 <attribute name="VALUE" x="85.09" y="46.99" size="1.778" layer="96" rot="R90"/>
 </instance>
-<instance part="VR2" gate="1" x="88.9" y="66.04" smashed="yes">
+<instance part="VR3" gate="1" x="88.9" y="66.04" smashed="yes">
 <attribute name="NAME" x="82.931" y="62.23" size="1.778" layer="95" rot="R90"/>
 <attribute name="VALUE" x="85.09" y="62.23" size="1.778" layer="96" rot="R90"/>
@@
 <attribute name="VALUE" x="41.91" y="62.23" size="1.778" layer="96" rot="R90"/>
 </instance>
-<instance part="VR3" gate="1" x="38.1" y="33.02" smashed="yes">
+<instance part="VR2" gate="1" x="38.1" y="33.02" smashed="yes">
 <attribute name="NAME" x="32.131" y="29.21" size="1.778" layer="95" rot="R90"/>
 <attribute name="VALUE" x="34.29" y="29.21" size="1.778" layer="96" rot="R90"/>
@@
 <pinref part="JP1" gate="A" pin="1"/>
 <wire x1="101.6" y1="53.34" x2="109.22" y2="53.34" width="0.1524" layer="91"/>
-<pinref part="VR2" gate="1" pin="S"/>
+<pinref part="VR3" gate="1" pin="S"/>
 <wire x1="93.98" y1="66.04" x2="101.6" y2="66.04" width="0.1524" layer="91"/>
 <wire x1="101.6" y1="66.04" x2="101.6" y2="53.34" width="0.1524" layer="91"/>
@@
 <segment>
 <pinref part="GND2" gate="1" pin="GND"/>
-<pinref part="VR3" gate="1" pin="A"/>
+<pinref part="VR2" gate="1" pin="A"/>
 <wire x1="38.1" y1="25.4" x2="38.1" y2="27.94" width="0.1524" layer="91"/>
 </segment>
@@
 <net name="N$4" class="0">
 <segment>
-<pinref part="VR3" gate="1" pin="S"/>
+<pinref part="VR2" gate="1" pin="S"/>
 <pinref part="P1" gate="/1" pin="A"/>
 <wire x1="43.18" y1="33.02" x2="45.72" y2="33.02" width="0.1524" layer="91"/>
@@
 <segment>
 <pinref part="P1" gate="/2" pin="E"/>
-<pinref part="VR2" gate="1" pin="A"/>
+<pinref part="VR3" gate="1" pin="A"/>
 <wire x1="88.9" y1="55.88" x2="88.9" y2="60.96" width="0.1524" layer="91"/>
 </segment>
