File: inverter-welder/concepts/08_magnum_power_vip_4000/improvements/current_setting_display/sch/schematic.sch (EAGLE design)
At the start: 7 parts, among them P1 1k

Commit message: [Welder] Small fixes in schematics.
Other:
- note added: "do czerwonego przewodu nastawy prądu"
- note removed: "do czerwonego przewódu nastawy prądu"
Changed lines of the file:
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@@
 <sheet>
 <plain>
-<text x="116.84" y="53.34" size="1.778" layer="97">do czerwonego przewódu nastawy prądu</text>
+<text x="116.84" y="53.34" size="1.778" layer="97">do czerwonego przewodu nastawy prądu</text>
 <text x="116.84" y="50.8" size="1.778" layer="97">do czarnego przewódu nastawy prądu</text>
 <text x="116.84" y="48.26" size="1.778" layer="97">do zielonego przewódu nastawy prądu</text>
